File: matrix.kicad_sch (KiCad schematic)
At the start: 94 parts, among them SW10 K08, SW11 K09, SW12 K0A, SW13 K0B, SW14 K0C, SW15 K10, SW16 K11, SW17 K12, SW18 K13, SW19 K14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

Commit message: add text
Parts:
- D1, D10, D11, D12, D13, D14, D15, D16, D17, D18, D19, D2, D20, D21, D22, D23, D24, D25, D26, D27, D28, D29, D3, D30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: footprint Diode_SMD:D_0603_1608Metric -> libs:D_0603_1608Metric
