File: CC45.kicad_pcb (KiCad board)
At the start: 2 copper layers, 247 x 80.8 mm, 123 parts, among them SW1 RESET, SW10 K08, SW11 K09, SW12 K0A, SW13 K0B, SW14 K0C, SW15 K10, SW16 K11, SW17 K12, SW18 K13, SW19 K14, SW2 K00, SW20 K15, SW21 K16, SW22 K17, SW23 K18, SW24 K19, SW25 K1A, SW26 K1B, SW27 K20, SW28 K21, SW29 K22, SW3 K01, SW30 K23, SW31 K24, SW32 K25, SW33 K26, SW34 K27, SW35 K28, SW36 K29, SW37 K2A, SW38 K2B, SW39 K30, SW4 K02, SW40 K31, SW41 K32, SW42 K33, SW43 K34, SW44 K36, SW45 K38, SW46 K39, SW47 K3A, SW48 K3B, SW5 K03, SW6 K04, SW7 K05, SW8 K06, SW9 K07, U1 ATmega32U4-AU, U2 PRTR5V0U2X, X1 XTAL

Commit message: routing
Parts:
- moved R1 44.4 mm to (247.0, 59.7), turned to -90 degrees
- moved R3 0.13 mm to (233.6, 57.2)
Routing:
- net /USB_N: track 7.68 -> 89.6 mm
- net /USB_P: track 7.66 -> 88.3 mm
- net Vcc: track 613.7 -> 661.5 mm, vias 27 -> 29
- net row0: track 274.3 -> 283.2 mm
- net row1: track 174.9 -> 181.8 mm
- net VCC: track 32.6 -> 26.9 mm
- net Net-(R1-Pad2): track 0.00 -> 3.26 mm
- net GND: track 711.5 -> 714.0 mm, vias 36 -> 37
- net Net-(D7-Pad2): track 7.23 -> 8.39 mm
- net Net-(D20-Pad2): track 19.7 -> 20.7 mm
- net Net-(D2-Pad2): track 4.97 -> 5.86 mm
- net Net-(D5-Pad2): track 4.88 -> 5.75 mm
- net Net-(SW11-Pad9): track 20.7 -> 21.6 mm
- net Net-(D19-Pad2): track 4.71 -> 5.43 mm
- net Net-(R6-Pad2): track 4.92 -> 5.62 mm

Commit message: fix drc
Parts:
- moved R4 90.3 mm to (238.5, 44.8), turned to 180 degrees
- moved SW1 84.1 mm to (234.4, 40.2), turned to 180 degrees
Routing:
- net col0: track 48.6 -> 70.0 mm
- net RESET: track 0.00 -> 20.4 mm, vias 0 -> 2
- net Vcc: track 661.5 -> 674.6 mm, vias 29 -> 30
- net GND: track 714.0 -> 720.5 mm, vias 37 -> 38
- net Net-(D26-Pad2): track 5.11 -> 0.00 mm
- net Net-(D7-Pad2): track 8.39 -> 7.03 mm
- net row1: track 181.8 -> 180.8 mm
- net row0: track 283.2 -> 282.3 mm
- net Net-(D20-Pad2): track 20.7 -> 19.9 mm
- net Net-(D8-Pad2): track 26.7 -> 26.0 mm

Commit message: routing lol
Parts:
- moved C1 73.8 mm to (233.6, 61.1)
- moved C2 1.97 mm to (245.9, 53.4)
- moved F1 1.21 mm to (157.6, 41.1), turned to 180 degrees
- moved R1 1.04 mm to (246.3, 60.4), turned to 180 degrees
- moved C5 0.36 mm to (232.9, 54.6), turned to 180 degrees
- turned SW32 to 0 degrees
Connections:
- SW17 pad 1: Net-(SW17-Pad1) -> col2
- SW26 pad 9: (no net) -> Net-(SW26-Pad9)
- SW27 pad 1: Net-(D26-Pad2) -> col0
- SW27 pad 10: (no net) -> Vcc
- SW27 pad 11: (no net) -> Net-(SW26-Pad9)
- SW27 pad 12: (no net) -> GND
- SW27 pad 2: col0 -> Net-(D26-Pad2)
- SW27 pad 9: (no net) -> Net-(SW27-Pad9)
- SW28 pad 1: Net-(D27-Pad2) -> col1
- SW28 pad 10: (no net) -> Vcc
- SW28 pad 11: (no net) -> Net-(SW27-Pad9)
- SW28 pad 12: (no net) -> GND
- SW28 pad 2: col1 -> Net-(D27-Pad2)
- SW28 pad 9: (no net) -> Net-(SW28-Pad9)
- SW29 pad 1: Net-(D28-Pad2) -> col2
- SW29 pad 10: (no net) -> Vcc
- SW29 pad 11: (no net) -> Net-(SW28-Pad9)
- SW29 pad 12: (no net) -> GND
- SW29 pad 2: col2 -> Net-(D28-Pad2)
- SW29 pad 9: (no net) -> Net-(SW29-Pad9)
- SW30 pad 1: Net-(D29-Pad2) -> col3
- SW30 pad 10: (no net) -> Vcc
- SW30 pad 11: (no net) -> Net-(SW29-Pad9)
- SW30 pad 12: (no net) -> GND
- SW30 pad 2: col3 -> Net-(D29-Pad2)
- SW30 pad 9: (no net) -> Net-(SW30-Pad9)
- SW31 pad 1: Net-(D30-Pad2) -> col4
- SW31 pad 10: (no net) -> Vcc
- SW31 pad 11: (no net) -> Net-(SW30-Pad9)
- SW31 pad 12: (no net) -> GND
- SW31 pad 2: col4 -> Net-(D30-Pad2)
- SW31 pad 9: (no net) -> Net-(SW31-Pad9)
- SW32 pad 1: Net-(D31-Pad2) -> col5
- SW32 pad 10: (no net) -> Vcc
- SW32 pad 11: (no net) -> Net-(SW31-Pad9)
- SW32 pad 12: (no net) -> GND
- SW32 pad 2: col5 -> Net-(D31-Pad2)
- SW32 pad 9: (no net) -> Net-(SW32-Pad9)
- SW33 pad 1: Net-(D32-Pad2) -> col6
- SW33 pad 10: (no net) -> Vcc
- SW33 pad 11: (no net) -> Net-(SW32-Pad9)
- SW33 pad 12: (no net) -> GND
- SW33 pad 2: col6 -> Net-(D32-Pad2)
- SW33 pad 9: (no net) -> Net-(SW33-Pad9)
- SW34 pad 1: Net-(D33-Pad2) -> col7
- SW34 pad 10: (no net) -> Vcc
- SW34 pad 11: (no net) -> Net-(SW33-Pad9)
- SW34 pad 12: (no net) -> GND
- SW34 pad 2: col7 -> Net-(D33-Pad2)
- SW34 pad 9: (no net) -> Net-(SW34-Pad9)
- SW35 pad 1: Net-(D34-Pad2) -> col8
- SW35 pad 10: (no net) -> Vcc
- SW35 pad 11: (no net) -> Net-(SW34-Pad9)
- SW35 pad 12: (no net) -> GND
- SW35 pad 2: col8 -> Net-(D34-Pad2)
- SW35 pad 9: (no net) -> Net-(SW35-Pad9)
- SW36 pad 1: Net-(D35-Pad2) -> col9
- SW36 pad 10: (no net) -> Vcc
- SW36 pad 11: (no net) -> Net-(SW35-Pad9)
- SW36 pad 12: (no net) -> GND
- SW36 pad 2: col9 -> Net-(D35-Pad2)
- SW36 pad 9: (no net) -> Net-(SW36-Pad9)
- SW37 pad 1: Net-(D36-Pad2) -> col10
- SW37 pad 10: (no net) -> Vcc
- SW37 pad 11: (no net) -> Net-(SW36-Pad9)
- SW37 pad 12: (no net) -> GND
- SW37 pad 2: col10 -> Net-(D36-Pad2)
- SW37 pad 9: (no net) -> Net-(SW37-Pad9)
- SW38 pad 1: Net-(D37-Pad2) -> col11
- SW38 pad 10: (no net) -> Vcc
- SW38 pad 11: (no net) -> Net-(SW37-Pad9)
- SW38 pad 12: (no net) -> GND
- SW38 pad 2: col11 -> Net-(D37-Pad2)
- SW4 pad 1: Net-(SW17-Pad1) -> col2
- U1 pad 1: col7 -> col10
- U1 pad 12: col6 -> col11
- U1 pad 27: col0 -> col4
- U1 pad 28: row2 -> col3
- U1 pad 30: col2 -> row2
- U1 pad 31: col3 -> col0
- U1 pad 32: col4 -> col2
- U1 pad 36: col5 -> col12
- U1 pad 37: col8 -> col6
- U1 pad 38: col9 -> col7
- U1 pad 39: col10 -> col8
- U1 pad 40: col11 -> col9
- U1 pad 41: col12 -> col5
Routing:
- net row2: track 0.00 -> 325.2 mm, vias 0 -> 4
- net Vcc: track 674.6 -> 993.3 mm, vias 30 -> 47
- net GND: track 720.5 -> 1029.9 mm, vias 38 -> 51
- net Net-(SW14-Pad9): track 0.00 -> 262.4 mm, vias 0 -> 4
- net Net-(SW26-Pad9): track 0.00 -> 257.0 mm, vias 0 -> 2
- net col2: track 0.00 -> 235.4 mm, vias 0 -> 5
- net col0: track 70.0 -> 285.4 mm, vias 0 -> 4
- net col1: track 57.1 -> 257.3 mm, vias 4 -> 5
- net col4: track 21.0 -> 206.3 mm, vias 2 -> 5
- net col3: track 56.0 -> 224.5 mm, vias 4 -> 6
- net col6: track 19.0 -> 155.5 mm, vias 1 -> 5
- net col5: track 53.5 -> 162.1 mm, vias 4 -> 5
- net row1: track 180.8 -> 289.2 mm, vias 9 -> 15
- net col7: track 30.6 -> 137.3 mm, vias 2 -> 5
- net col8: track 14.6 -> 118.1 mm, vias 1 -> 5
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
Commit message: routing lmao
Parts:
- moved D42 27.1 mm to (140.2, 88.3)
- moved D46 4.15 mm to (244.3, 86.4)
- moved D39 2.24 mm to (69.4, 92.4)
- moved D38 1.86 mm to (45.9, 88.4)
- moved D45 1.27 mm to (224.2, 91.5)
- moved D40 1.24 mm to (93.2, 91.5)
- moved D44 0.74 mm to (200.4, 90.9)
- turned SW44 to 180 degrees
Connections:
- SW38 pad 9: (no net) -> Net-(SW38-Pad9)
- SW39 pad 1: Net-(D38-Pad2) -> col0 (x2)
- SW39 pad 10: (no net) -> Vcc (x2)
- SW39 pad 11: (no net) -> Net-(SW38-Pad9) (x2)
- SW39 pad 12: (no net) -> GND (x2)
- SW39 pad 2: col0 -> Net-(D38-Pad2) (x2)
- SW39 pad 9: (no net) -> Net-(SW39-Pad9) (x2)
- SW40 pad 1: Net-(D39-Pad2) -> col1 (x2)
- SW40 pad 10: (no net) -> Vcc (x2)
- SW40 pad 11: (no net) -> Net-(SW39-Pad9) (x2)
- SW40 pad 12: (no net) -> GND (x2)
- SW40 pad 2: col1 -> Net-(D39-Pad2) (x2)
- SW40 pad 9: (no net) -> Net-(SW40-Pad9) (x2)
- SW41 pad 1: Net-(D40-Pad2) -> col2 (x2)
- SW41 pad 10: (no net) -> Vcc (x2)
- SW41 pad 11: (no net) -> Net-(SW40-Pad9) (x2)
- SW41 pad 12: (no net) -> GND (x2)
- SW41 pad 2: col2 -> Net-(D40-Pad2) (x2)
- SW41 pad 9: (no net) -> Net-(SW41-Pad9) (x2)
- SW42 pad 1: Net-(D41-Pad2) -> col3
- SW42 pad 10: (no net) -> Vcc
- SW42 pad 11: (no net) -> Net-(SW41-Pad9)
- SW42 pad 12: (no net) -> GND
- SW42 pad 2: col3 -> Net-(D41-Pad2)
- SW42 pad 9: (no net) -> Net-(SW42-Pad9)
- SW43 pad 1: Net-(D42-Pad2) -> col4 (x2)
- SW43 pad 10: (no net) -> Vcc (x2)
- SW43 pad 11: (no net) -> Net-(SW42-Pad9) (x2)
- SW43 pad 12: (no net) -> GND (x2)
- SW43 pad 2: col4 -> Net-(D42-Pad2) (x2)
- SW43 pad 9: (no net) -> Net-(SW43-Pad9) (x2)
- SW44 pad 1: Net-(D43-Pad2) -> col6 (x3)
- SW44 pad 10: Net-(SW44-Pad10) -> Vcc (x3)
- SW44 pad 11: Net-(SW44-Pad11) -> Net-(SW43-Pad9) (x3)
- SW44 pad 12: Net-(SW44-Pad12) -> GND (x3)
- SW44 pad 2: col6 -> Net-(D43-Pad2) (x3)
- SW45 pad 1: Net-(D44-Pad2) -> col8
- SW45 pad 10: (no net) -> Vcc
- SW45 pad 12: (no net) -> GND
- SW45 pad 2: col8 -> Net-(D44-Pad2)
- SW45 pad 9: (no net) -> Net-(SW45-Pad9)
- SW46 pad 1: Net-(D45-Pad2) -> col9 (x2)
- SW46 pad 10: (no net) -> Vcc (x2)
- SW46 pad 11: (no net) -> Net-(SW45-Pad9) (x2)
- SW46 pad 12: (no net) -> GND (x2)
- SW46 pad 2: col9 -> Net-(D45-Pad2) (x2)
- SW46 pad 9: (no net) -> Net-(SW46-Pad9) (x2)
- SW47 pad 1: Net-(D46-Pad2) -> col10 (x2)
- SW47 pad 10: (no net) -> Vcc (x2)
- SW47 pad 11: (no net) -> Net-(SW46-Pad9) (x2)
- SW47 pad 12: (no net) -> GND (x2)
- SW47 pad 2: col10 -> Net-(D46-Pad2) (x2)
- SW47 pad 9: (no net) -> Net-(SW47-Pad9) (x2)
- SW48 pad 1: Net-(D47-Pad2) -> col11 (x2)
- SW48 pad 10: (no net) -> Vcc (x2)
- SW48 pad 11: (no net) -> Net-(SW47-Pad9) (x2)
- SW48 pad 12: (no net) -> GND (x2)
- SW48 pad 2: col11 -> Net-(D47-Pad2) (x2)
- SW48 pad 9: (no net) -> Net-(SW48-Pad9) (x2)
Routing:
- net GND: track 1029.9 -> 1303.3 mm, vias 51 -> 67
- net Net-(SW38-Pad9): track 0.00 -> 264.6 mm, vias 0 -> 5
- net row3: track 54.8 -> 295.4 mm, vias 1 -> 7
- net Vcc: track 993.3 -> 1228.8 mm, vias 47 -> 62
- net Net-(SW43-Pad9): track 0.00 -> 80.2 mm, vias 0 -> 6
- net Net-(SW39-Pad9): track 0.00 -> 68.0 mm, vias 0 -> 4
- net Net-(SW44-Pad9): track 0.00 -> 48.4 mm, vias 0 -> 2
- net Net-(D43-Pad2): track 0.00 -> 47.3 mm
- net Net-(SW40-Pad9): track 0.00 -> 39.6 mm, vias 0 -> 4
- net col6: track 155.5 -> 193.4 mm, vias 5 -> 7
- net col1: track 257.3 -> 291.1 mm, vias 5 -> 7
- net col4: track 206.3 -> 237.8 mm, vias 5 -> 7
- net Net-(SW42-Pad9): track 0.00 -> 31.3 mm, vias 0 -> 2
- net Net-(SW41-Pad9): track 0.00 -> 27.4 mm, vias 0 -> 2
- net col2: track 235.4 -> 262.2 mm, vias 5 -> 7
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
Commit message: finish routing + zoning
Parts:
- moved D44 0.72 mm to (200.4, 91.6)
Routing:
- net Vcc: track 1228.8 -> 1364.0 mm, vias 62 -> 69
- net row3: track 295.4 -> 406.9 mm, vias 7 -> 11
- net GND: track 1303.3 -> 1365.6 mm, vias 67 -> 75
- net Net-(SW46-Pad9): track 0.00 -> 55.9 mm, vias 0 -> 4
- net Net-(SW47-Pad9): track 0.00 -> 52.9 mm
- net col10: track 57.2 -> 92.2 mm, vias 6 -> 8
- net col11: track 93.3 -> 122.4 mm, vias 4 -> 8
- net Net-(SW45-Pad9): track 0.00 -> 27.1 mm, vias 0 -> 2
- net Net-(SW21-Pad9): track 0.00 -> 19.7 mm, vias 0 -> 2
- net col9: track 100.9 -> 117.2 mm, vias 5 -> 8
- net Net-(D46-Pad2): track 0.00 -> 13.7 mm
- net Net-(D47-Pad2): track 0.00 -> 9.92 mm
- net Net-(D44-Pad2): track 5.78 -> 6.48 mm
- added copper zone on F.Cu, net GND

Commit message: moar zoning
Routing:
- added copper zone on B.Cu, net Vcc
Changed lines of the file:
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@@
+    )
+  )
+  (zone (net 100) (net_name "Vcc") (layer "B.Cu") (hatch edge 0.508)
+    (connect_pads (clearance 0.508))
+    (min_thickness 0.254)
+    (fill yes (thermal_gap 0.508) (thermal_bridge_width 0.508))
+    (polygon
+      (pts
+        (xy 281.1272 23.0632) (xy 279.908 107.7468) (xy 236.4232 137.3124) (xy -14.2748 130.7084) (xy -7.9756 22.0472)
+        (xy 85.5472 -0.3048)
+      )
     )
   )

Commit message: finishing touches
Routing:
- net Net-(SW48-Pad9): track 0.00 -> 26.3 mm, vias 0 -> 2
- net GND: track 1365.6 -> 1379.8 mm
- net Net-(SW43-Pad9): track 80.2 -> 82.5 mm
- removed copper zone on B.Cu, net GND

Commit message: doot
Other:
- board text removed: "JLCJLCJLCJLC"
