File: CC45.kicad_pcb (KiCad board)
At the start: 2 copper layers, 247 x 80.8 mm, 123 parts, among them SW1 RESET, SW10 K08, SW11 K09, SW12 K0A, SW13 K0B, SW14 K0C, SW15 K10, SW16 K11, SW17 K12, SW18 K13, SW19 K14, SW2 K00, SW20 K15, SW21 K16, SW22 K17, SW23 K18, SW24 K19, SW25 K1A, SW26 K1B, SW27 K20, SW28 K21, SW29 K22, SW3 K01, SW30 K23, SW31 K24, SW32 K25, SW33 K26, SW34 K27, SW35 K28, SW36 K29, SW37 K2A, SW38 K2B, SW39 K30, SW4 K02, SW40 K31, SW41 K32, SW42 K33, SW43 K34, SW44 K36, SW45 K38, SW46 K39, SW47 K3A, SW48 K3B, SW5 K03, SW6 K04, SW7 K05, SW8 K06, SW9 K07, U1 ATmega32U4-AU, U2 PRTR5V0U2X, X1 XTAL

Commit message: add text
Other:
- board text added: "CC45 RGB"
- board text added: "Designed in Kicad"
- board text added: "HID Technologies"
- board text added: "Limited edition prototype"
- board text added: "Not intended for commercial use"
- board text added: "Original design by Druz"
- board text added: "Rev 1.0"

Commit message: add vias in MCU
Routing:
- net /USB_N: track 106.6 -> 106.1 mm
- net (no net): vias 0 -> 5
Changed lines of the file:
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@@
     (thickness 1.6)
     (drawings 22)
-    (tracks 2842)
+    (tracks 2843)
     (modules 123)
     (nets 126)
@@
       (dielectric_constraints no)
     )
-    (last_trace_width 0.2)
+    (last_trace_width 0.25)
     (user_trace_width 0.2)
     (user_trace_width 0.3)
@@
       (effects (font (size 1 1) (thickness 0.15)) (justify mirror))
     )
+    (fp_line (start 0.8 0.4) (end -0.5 0.4) (layer "B.Fab") (width 0.1))
+    (fp_line (start -0.5 0.4) (end -0.8 0.1) (layer "B.Fab") (width 0.1))
+    (fp_line (start -0.8 0.1) (end -0.8 -0.4) (layer "B.Fab") (width 0.1))
+    (fp_line (start -0.8 -0.4) (end 0.8 -0.4) (layer "B.Fab") (width 0.1))
+    (fp_line (start 0.8 -0.4) (end 0.8 0.4) (layer "B.Fab") (width 0.1))
+    (fp_line (start 0.8 0.735) (end -1.485 0.735) (layer "B.SilkS") (width 0.12))
+    (fp_line (start -1.485 0.735) (end -1.485 -0.735) (layer "B.SilkS") (width 0.12))
+    (fp_line (start -1.485 -0.735) (end 0.8 -0.735) (layer "B.SilkS") (width 0.12))
+    (fp_line (start -1.48 -0.73) (end -1.48 0.73) (layer "B.CrtYd") (width 0.05))
+    (fp_line (start -1.48 0.73) (end 1.48 0.73) (layer "B.CrtYd") (width 0.05))
+    (fp_line (start 1.48 0.73) (end 1.48 -0.73) (layer "B.CrtYd") (width 0.05))
+    (fp_line (start 1.48 -0.73) (end -1.48 -0.73) (layer "B.CrtYd") (width 0.05))
     (fp_text user "${REFERENCE}" (at 0 0 270) (layer "B.Fab")
       (effects (font (size 0.4 0.4) (thickness 0.06)) (justify mirror))
     )
-    (fp_line (start 1.48 -0.73) (end -1.48 -0.73) (layer "B.CrtYd") (width 0.05))
-    (fp_line (start 1.48 0.73) (end 1.48 -0.73) (layer "B.CrtYd") (width 0.05))
-    (fp_line (start -1.48 0.73) (end 1.48 0.73) (layer "B.CrtYd") (width 0.05))
-    (fp_line (start -1.48 -0.73) (end -1.48 0.73) (layer "B.CrtYd") (width 0.05))
-    (fp_line (start -1.485 -0.735) (end 0.8 -0.735) (layer "B.SilkS") (width 0.12))
-    (fp_line (start -1.485 0.735) (end -1.485 -0.735) (layer "B.SilkS") (width 0.12))
-    (fp_line (start 0.8 0.735) (end -1.485 0.735) (layer "B.SilkS") (width 0.12))
-    (fp_line (start 0.8 -0.4) (end 0.8 0.4) (layer "B.Fab") (width 0.1))
-    (fp_line (start -0.8 -0.4) (end 0.8 -0.4) (layer "B.Fab") (width 0.1))
-    (fp_line (start -0.8 0.1) (end -0.8 -0.4) (layer "B.Fab") (width 0.1))
-    (fp_line (start -0.5 0.4) (end -0.8 0.1) (layer "B.Fab") (width 0.1))
-    (fp_line (start 0.8 0.4) (end -0.5 0.4) (layer "B.Fab") (width 0.1))
-    (pad "2" smd roundrect (at 0.7875 0 90) (size 0.875 0.95) (layers "B.Cu" "B.Paste" "B.Mask") (roundrect_rratio 0.25)
-      (net 52 "Net-(D46-Pad2)") (pinfunction "A"))
     (pad "1" smd roundrect (at -0.7875 0 90) (size 0.875 0.95) (layers "B.Cu" "B.Paste" "B.Mask") (roundrect_rratio 0.25)
       (net 44 "row3") (pinfunction "K"))
+    (pad "2" smd roundrect (at 0.7875 0 90) (size 0.875 0.95) (layers "B.Cu" "B.Paste" "B.Mask") (roundrect_rratio 0.25)
+      (net 52 "Net-(D46-Pad2)") (pinfunction "A"))
     (model "${KISYS3DMOD}/Diode_SMD.3dshapes/D_0603_1608Metric.wrl"
       (at (xyz 0 0 0))
@@
     (fp_line (start -1.6 0.8) (end 1.6 0.8) (layer "B.Fab") (width 0.1))
     (fp_line (start -1.6 -0.8) (end -1.6 0.8) (layer "B.Fab") (width 0.1))
-    (pad "2" smd roundrect (at 1.4875 0 180) (size 1.425 1.75) (layers "B.Cu" "B.Paste" "B.Mask") (roundrect_rratio 0.175439)
+    (pad "2" smd roundrect (at 1.4875 0 180) (size 1.425 1.75) (layers "B.Cu" "B.Paste" "B.Mask") (roundrect_rratio 0.175439298245614)
       (net 54 "VCC"))
-    (pad "1" smd roundrect (at -1.4875 0 180) (size 1.425 1.75) (layers "B.Cu" "B.Paste" "B.Mask") (roundrect_rratio 0.175439)
+    (pad "1" smd roundrect (at -1.4875 0 180) (size 1.425 1.75) (layers "B.Cu" "B.Paste" "B.Mask") (roundrect_rratio 0.175439298245614)
       (net 100 "Vcc"))
     (model "${KISYS3DMOD}/Fuse.3dshapes/Fuse_1206_3216Metric.wrl"
@@
   (gr_arc (start 24.9375 98.5625) (end 23.75 98.5625) (angle -90) (layer "Edge.Cuts") (width 0.15))
   (gr_arc (start 24.9375 24.9375) (end 24.9375 23.75) (angle -90) (layer "Edge.Cuts") (width 0.15))
+  (segment (start 243.2304 87.5792) (end 244.86 89.2088) (width 0.2) (layer "B.Cu") (net 52))
+  (segment (start 243.2304 86.6648) (end 243.2304 87.5792) (width 0.2) (layer "B.Cu") (net 52))
+  (segment (start 244.2972 85.598) (end 243.2304 86.6648) (width 0.2) (layer "B.Cu") (net 52))
+  (segment (start 243.8692 85.17) (end 244.2972 85.598) (width 0.2) (layer "B.Cu") (net 52))
+  (segment (start 238.84 85.17) (end 243.8692 85.17) (width 0.2) (layer "B.Cu") (net 52))
+  (segment (start 244.86 89.2088) (end 244.86 92.79) (width 0.2) (layer "B.Cu") (net 52))
+  (segment (start 247.3452 80.264) (end 247.3452 84.125) (width 0.2) (layer "B.Cu") (net 44) (status 8000))
+  (segment (start 247.3452 84.125) (end 244.2972 87.173) (width 0.2) (layer "B.Cu") (net 44) (status 8000))
+  (via (at 242.7224 57.023) (size 0.8) (drill 0.4) (layers "F.Cu" "B.Cu") (net 0))
+  (via (at 240.9444 58.547) (size 0.8) (drill 0.4) (layers "F.Cu" "B.Cu") (net 0))
+  (via (at 239.1664 57.023) (size 0.8) (drill 0.4) (layers "F.Cu" "B.Cu") (net 0))
+  (via (at 242.7224 54.483) (size 0.8) (drill 0.4) (layers "F.Cu" "B.Cu") (net 0))
+  (via (at 239.0394 54.61) (size 0.8) (drill 0.4) (layers "F.Cu" "B.Cu") (net 0))
+  (segment (start 224.7392 45.2628) (end 230.378 50.9016) (width 0.2) (layer "B.Cu") (net 73))
+  (segment (start 160.6296 45.2628) (end 224.7392 45.2628) (width 0.2) (layer "B.Cu") (net 73))
+  (segment (start 157.656579 42.289779) (end 160.6296 45.2628) (width 0.2) (layer "B.Cu") (net 73))
+  (segment (start 156.988 29.276) (end 157.656579 29.944579) (width 0.2) (layer "B.Cu") (net 73))
+  (segment (start 230.378 56.1342) (end 232.9178 58.674) (width 0.2) (layer "B.Cu") (net 73))
+  (segment (start 157.656579 29.944579) (end 157.656579 42.289779) (width 0.2) (layer "B.Cu") (net 73))
+  (segment (start 230.378 50.9016) (end 230.378 56.1342) (width 0.2) (layer "B.Cu") (net 73))
   (via (at 266.3952 92.6592) (size 0.8) (drill 0.4) (layers "F.Cu" "B.Cu") (net 125))
   (segment (start 264.5156 86.8172) (end 262.9916 86.8172) (width 0.2) (layer "F.Cu") (net 125))
@@
   (segment (start 165.0492 92.761798) (end 165.0492 94.5388) (width 0.2) (layer "B.Cu") (net 75))
   (segment (start 166.2684 91.542598) (end 165.0492 92.761798) (width 0.2) (layer "B.Cu") (net 75))
-  (segment (start 243.2304 86.6648) (end 243.2304 87.5792) (width 0.2) (layer "B.Cu") (net 52))
-  (segment (start 244.2972 85.598) (end 243.2304 86.6648) (width 0.2) (layer "B.Cu") (net 52))
-  (segment (start 243.2304 87.5792) (end 244.86 89.2088) (width 0.2) (layer "B.Cu") (net 52))
-  (segment (start 244.86 89.2088) (end 244.86 92.79) (width 0.2) (layer "B.Cu") (net 52))
   (segment (start 201.2696 91.523583) (end 201.2696 90.424) (width 0.2) (layer "B.Cu") (net 44))
   (segment (start 200.355686 92.437497) (end 201.2696 91.523583) (width 0.2) (layer "B.Cu") (net 44))
@@
   (segment (start 268.6812 77.7748) (end 266.573 79.883) (width 0.2) (layer "F.Cu") (net 44) (status 8000))
   (via (at 247.3452 80.264) (size 0.8) (drill 0.4) (layers "F.Cu" "B.Cu") (net 44))
-  (segment (start 247.3452 84.125) (end 244.2972 87.173) (width 0.2) (layer "B.Cu") (net 44) (status 8000))
-  (segment (start 247.3452 80.264) (end 247.3452 84.125) (width 0.2) (layer "B.Cu") (net 44) (status 8000))
   (segment (start 202.721939 80.774535) (end 221.114585 80.774535) (width 0.3) (layer "F.Cu") (net 1))
   (via (at 223.9264 79.5528) (size 0.8) (drill 0.4) (layers "F.Cu" "B.Cu") (net 44))
@@
   (segment (start 167.4876 58.928) (end 169.2913 60.7317) (width 0.2) (layer "B.Cu") (net 95))
   (segment (start 169.2913 60.7317) (end 170.2375 60.7317) (width 0.2) (layer "B.Cu") (net 95))
-  (segment (start 238.84 85.17) (end 243.8692 85.17) (width 0.2) (layer "B.Cu") (net 52))
-  (segment (start 243.8692 85.17) (end 244.2972 85.598) (width 0.2) (layer "B.Cu") (net 52))
   (via (at 261.7724 87.4776) (size 0.8) (drill 0.4) (layers "F.Cu" "B.Cu") (net 100))
   (segment (start 261.7724 87.4776) (end 260.91708 87.4776) (width 0.3) (layer "B.Cu") (net 100))
@@
   (segment (start 239.319021 52.532501) (end 239.419 52.63248) (width 0.3) (layer "B.Cu") (net 100))
   (segment (start 236.3469 51.2064) (end 237.17191 52.03141) (width 0.3) (layer "B.Cu") (net 100))
-  (segment (start 156.988 29.276) (end 157.656579 29.944579) (width 0.2) (layer "B.Cu") (net 73))
-  (segment (start 230.378 50.9016) (end 224.7392 45.2628) (width 0.2) (layer "B.Cu") (net 73))
-  (segment (start 224.7392 45.2628) (end 160.6296 45.2628) (width 0.2) (layer "B.Cu") (net 73))
-  (segment (start 230.378 56.1342) (end 230.378 50.9016) (width 0.2) (layer "B.Cu") (net 73))
   (segment (start 230.778011 54.959411) (end 230.778011 50.742811) (width 0.2) (layer "B.Cu") (net 74))
-  (segment (start 157.656579 29.944579) (end 157.656579 39.515857) (width 0.2) (layer "B.Cu") (net 73))
-  (segment (start 232.9178 58.674) (end 230.378 56.1342) (width 0.2) (layer "B.Cu") (net 73))
-  (segment (start 160.6296 45.2628) (end 160.147 44.7802) (width 0.2) (layer "B.Cu") (net 73))
-  (segment (start 159.758236 44.7802) (end 160.147 44.7802) (width 0.2) (layer "B.Cu") (net 73))
   (segment (start 232.9178 57.0992) (end 230.778011 54.959411) (width 0.2) (layer "B.Cu") (net 74))
-  (segment (start 157.256568 42.278532) (end 159.758236 44.7802) (width 0.2) (layer "B.Cu") (net 73))
-  (segment (start 157.256568 39.915868) (end 157.256568 42.278532) (width 0.2) (layer "B.Cu") (net 73))
-  (segment (start 157.656579 39.515857) (end 157.256568 39.915868) (width 0.2) (layer "B.Cu") (net 73))
   (segment (start 161.335242 44.412778) (end 160.086632 43.164168) (width 0.3) (layer "B.Cu") (net 1))
   (segment (start 225.091289 44.412778) (end 161.335242 44.412778) (width 0.3) (layer "B.Cu") (net 1))
